File: wifi-light.sch (KiCad schematic (older format))
At the start: 26 parts, among them U1? SPX3819

Commit message: update
Parts:
- added C?: 1.0 uF, symbol CP
- added D? (x4): D, symbol D
- added F?: FUSE, symbol FUSE
- added Q?: DPAK, TO-220, symbol DPAK
- C?: value C -> 1.0uF
- C?: value C -> 100nF
Connections:
- net labels added: +12V, GND, VFB
- wire segments 0 -> 43
Other:
- moved on the sheet: C?, D?, R?, U1?, U?
